File: AZ1A_PCB_001/AZ1A_PCB_001.brd (EAGLE design)
At the start: 160 x 120 mm, 35 parts

Commit message: Actualización de PCB
Parts:
- moved CNC 87.7 mm to (165.8, 79.5), turned to 270 degrees
- moved EJEX 73.5 mm to (78.5, 83.9), turned to 270 degrees
- moved 12VDC 71.8 mm to (175.0, 33.6)
- moved 12VDC-PRINTER3D 64.2 mm to (175.0, 25.2)
- moved 12VDC-CNC 56.6 mm to (175.3, 42.1)
- moved LASER 55.8 mm to (165.8, 41.8), turned to 270 degrees
- moved EJES/CNC-LASER 52.6 mm to (131.8, 76.9)
- moved EJEY 50.3 mm to (86.3, 94.0), turned to 270 degrees
- moved CONECTOR-CNC/LASER 48.7 mm to (132.4, 60.1), turned to 180 degrees
- moved USB-CNC/LASER 46.0 mm to (154.3, 14.8)
- moved EJEAUX 41.4 mm to (78.3, 104.0), turned to 270 degrees
- moved USB 41.1 mm to (44.3, 41.8)
- moved EJES/PRINTER3D 35.1 mm to (31.3, 113.0), turned to 180 degrees
- moved CONECTOR-PRINTER3D 34.4 mm to (37.4, 8.74), turned to 180 degrees
- moved USB-PRINTER3D 29.4 mm to (32.7, 54.7)
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Routing:
- net N$47: track 0.00 -> 61.6 mm
- net N$48: track 0.00 -> 57.4 mm
- net N$49: track 0.00 -> 53.3 mm
- net N$50: track 0.00 -> 49.1 mm
- net N$51: track 0.00 -> 45.0 mm
- net N$52: track 0.00 -> 40.8 mm
- net N$53: track 0.00 -> 36.7 mm
- net N$6: track 0.00 -> 36.5 mm
- net N$54: track 0.00 -> 32.8 mm
- net N$21: track 0.00 -> 32.3 mm
- net N$57: track 0.00 -> 28.6 mm
- net N$24: track 0.00 -> 27.9 mm
- net N$14: track 0.00 -> 27.0 mm
- net N$13: track 0.00 -> 26.6 mm
- net N$15: track 0.00 -> 26.6 mm
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Other:
- board size 160 x 120 mm -> 180 x 125 mm

Commit message: Actualización PCB casi finalizando la PCB
Parts:
- added JP1, JP2: (no value), pinhead:1X01
- added JP3, JP4: (no value), pinhead:1X03
- moved LED-LASER 262.8 mm to (159.5, 13.4)
- moved R3 254.5 mm to (157.1, 19.3), turned to 180 degrees
- moved LED-CNC 233.7 mm to (117.8, 13.2)
- moved R2 182.6 mm to (80.7, 11.0), turned to 270 degrees
- moved 12VDC 149.5 mm to (25.5, 35.1)
- moved 12VDC-PRINTER3D 149.0 mm to (26.0, 25.7)
- moved 12VDC-LASER 105.3 mm to (154.5, 11.3)
- moved 12VDC-CNC 67.5 mm to (117.7, 7.16), turned to 0 degrees
- moved USB-CNC/LASER 65.7 mm to (120.8, 71.3)
- moved USB 49.0 mm to (83.8, 70.8)
- moved CONECTOR-PRINTER3D 33.4 mm to (48.7, 40.1), turned to 90 degrees
- moved CONECTOR-LASER 24.5 mm to (156.5, 34.7), turned to 270 degrees
- moved CONECTOR-CNC/LASER 20.2 mm to (135.6, 40.1), turned to 90 degrees
- moved USB-PRINTER3D 15.0 mm to (32.2, 69.7)
- moved LED-PRINTER3D 11.7 mm to (39.0, 25.9)
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Connections:
- removed net N$20: 12VDC-CNC.2, 12VDC-LASER.2, LED-CNC.2, LED-LASER.2, USB-CNC/LASER.4
- new net N$148: JP1.1, USB-CNC/LASER.4
- new net N$149: CNC/LASER-2.2, CNC/LASER-2.4, CNC/LASER-2.6, JP3.1, JP3.2, JP3.3
- net N$110: now also 12VDC-CNC.2, 12VDC-LASER.2, JP2.1, LED-CNC.2, LED-LASER.2
- net N$122: now also JP4.1, JP4.2, JP4.3; no longer CNC/LASER-2.2, CNC/LASER-2.4, CNC/LASER-2.6
Routing:
- net N$76: track 0.00 -> 877.8 mm
- net N$110: track 0.00 -> 518.8 mm
- net N$75: track 0.00 -> 354.0 mm
- net N$18: track 0.00 -> 203.7 mm
- net N$122: track 0.00 -> 180.8 mm
- net N$17: track 26.6 -> 203.9 mm
- net N$19: track 0.00 -> 172.8 mm
- net N$85: track 0.00 -> 162.2 mm
- net N$83: track 0.00 -> 160.0 mm
- net N$149: track 0.00 -> 154.8 mm
- net N$84: track 0.00 -> 131.9 mm
- net N$88: track 0.00 -> 111.5 mm
- net N$82: track 0.00 -> 105.7 mm
- net N$89: track 0.00 -> 101.8 mm
- net N$86: track 0.00 -> 100.2 mm
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Other:
- board size 180 x 125 mm -> 185 x 125 mm

Commit message: Actualizacion de PCB y dimensiones de Arduino UNO y MEGA
Parts:
- added JP10, JP13, JP14, JP9: (no value), pinhead:1X05
- added JP11, JP12, JP5, JP6: (no value), pinhead:1X02
- added JP15, JP16, JP7, JP8: (no value), pinhead:1X03
- moved 12VDC 32.8 mm to (19.7, 67.4)
- moved R3 1.84 mm to (158.4, 20.6)
Connections:
- new net N$153: CNC.15, JP10.1
- new net N$154: 12VDC-PRINTER3D.1, 12VDC.2, JP6.1, JP6.2, LED-PRINTER3D.1, USB-PRINTER3D.1
- new net N$155: 12VDC.1, JP7.1, JP7.2, JP7.3
- new net N$156: CNC.17, JP10.2
- new net N$157: CNC.19, JP10.3
- new net N$158: CNC.21, JP10.4
- new net N$159: CNC.23, JP10.5
- new net N$160: 12VDC-LASER.1, JP11.1, JP11.2, R3.2
- new net N$161: JP13.1, LASER.16
- new net N$162: JP13.2, LASER.18
- new net N$163: JP13.3, LASER.20
- new net N$164: JP13.4, LASER.22
- new net N$165: JP13.5, LASER.24
- new net N$166: JP15.1, JP15.2, JP15.3, LASER.10, LASER.12, LASER.14
- net N$106: now also JP9.4; no longer CNC.21
- net N$107: now also JP9.5; no longer CNC.23
- net N$108: now also JP12.1, JP12.2; no longer 12VDC-LASER.1, R3.2
- net N$110: now also JP5.1, JP5.2; no longer 12VDC-PRINTER3D.1, 12VDC.2, LED-PRINTER3D.1, USB-PRINTER3D.1
- net N$122: now also JP16.1, JP16.2, JP16.3; no longer LASER.10, LASER.12, LASER.14
- net N$17: now also JP8.1, JP8.2, JP8.3; no longer 12VDC.1
- net N$83: now also JP14.1; no longer LASER.16
- net N$84: now also JP14.2; no longer LASER.18
- net N$85: now also JP14.3; no longer LASER.20
- net N$86: now also JP14.4; no longer LASER.22
- net N$87: now also JP14.5; no longer LASER.24
- net N$88: now also JP9.1; no longer CNC.15
- net N$89: now also JP9.2; no longer CNC.17
- net N$90: now also JP9.3; no longer CNC.19
Routing:
- net N$154: track 0.00 -> 1458.5 mm
- net N$167: track 0.00 -> 173.3 mm
- net N$122: track 180.8 -> 344.6 mm
- net N$108: track 7.18 -> 163.1 mm
- net N$84: track 131.9 -> 6.20 mm
- net N$169: track 0.00 -> 120.1 mm
- net N$170: track 0.00 -> 120.0 mm
- net N$155: track 0.00 -> 107.2 mm
- net N$160: track 0.00 -> 74.8 mm
- net N$151: track 0.00 -> 71.1 mm
- net N$110: track 518.8 -> 449.3 mm
- net N$166: track 0.00 -> 69.1 mm
- net N$150: track 0.00 -> 68.6 mm
- net N$171: track 0.00 -> 61.1 mm
- net N$168: track 0.00 -> 61.0 mm
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