File: AZ1A_PCB_001/AZ1A_PCB_001.sch (EAGLE design)
At the start: 35 parts

Commit message: Actualización PCB casi finalizando la PCB
Parts:
- added JP1, JP2: (no value), pinhead:PINHD-1X1
- added JP3, JP4: (no value), pinhead:PINHD-1X3
Connections:
- removed net N$20: 12VDC-CNC.2, 12VDC-LASER.2, LED-CNC.2, LED-LASER.2, USB-CNC/LASER.4
- new net N$148: JP1.1, USB-CNC/LASER.4
- new net N$149: CNC/LASER-2.2, CNC/LASER-2.4, CNC/LASER-2.6, JP3.1, JP3.2, JP3.3
- net N$110: now also 12VDC-CNC.2, 12VDC-LASER.2, JP2.1, LED-CNC.2, LED-LASER.2
- net N$122: now also JP4.1, JP4.2, JP4.3; no longer CNC/LASER-2.2, CNC/LASER-2.4, CNC/LASER-2.6

Commit message: Actualizacion de PCB y dimensiones de Arduino UNO y MEGA
Parts:
- added JP10, JP13, JP14, JP9: (no value), pinhead:PINHD-1X5
- added JP11, JP12, JP5, JP6: (no value), pinhead:PINHD-1X2
- added JP15, JP16, JP7, JP8: (no value), pinhead:PINHD-1X3
Connections:
- new net N$153: CNC.15, JP10.1
- new net N$154: 12VDC-PRINTER3D.1, 12VDC.2, JP6.1, JP6.2, LED-PRINTER3D.1, USB-PRINTER3D.1
- new net N$155: 12VDC.1, JP7.1, JP7.2, JP7.3
- new net N$156: CNC.17, JP10.2
- new net N$157: CNC.19, JP10.3
- new net N$158: CNC.21, JP10.4
- new net N$159: CNC.23, JP10.5
- new net N$160: 12VDC-LASER.1, JP11.1, JP11.2, R3.2
- new net N$161: JP13.1, LASER.16
- new net N$162: JP13.2, LASER.18
- new net N$163: JP13.3, LASER.20
- new net N$164: JP13.4, LASER.22
- new net N$165: JP13.5, LASER.24
- new net N$166: JP15.1, JP15.2, JP15.3, LASER.10, LASER.12, LASER.14
- net N$106: now also JP9.4; no longer CNC.21
- net N$107: now also JP9.5; no longer CNC.23
- net N$108: now also JP12.1, JP12.2; no longer 12VDC-LASER.1, R3.2
- net N$110: now also JP5.1, JP5.2; no longer 12VDC-PRINTER3D.1, 12VDC.2, LED-PRINTER3D.1, USB-PRINTER3D.1
- net N$122: now also JP16.1, JP16.2, JP16.3; no longer LASER.10, LASER.12, LASER.14
- net N$17: now also JP8.1, JP8.2, JP8.3; no longer 12VDC.1
- net N$83: now also JP14.1; no longer LASER.16
- net N$84: now also JP14.2; no longer LASER.18
- net N$85: now also JP14.3; no longer LASER.20
- net N$86: now also JP14.4; no longer LASER.22
- net N$87: now also JP14.5; no longer LASER.24
- net N$88: now also JP9.1; no longer CNC.15
- net N$89: now also JP9.2; no longer CNC.17
- net N$90: now also JP9.3; no longer CNC.19
